File: PCB/memmert_pcb/memmert_pcb.kicad_sch (KiCad schematic)
At the start: 0 parts

Commit message: Deleted project library. Started editing schematic
Parts:
- added C1, C2: 100 nF, Capacitor_SMD:C_0603_1608Metric, symbol USER_Capacitors:100 nF
- added U1: PIC24FJXXXGL405_I_PT, USER_fp:TQFP48_PT_MCH, symbol USER_Microchip_PIC:PIC24FJXXXGL405_I_PT
Connections:
- new net +3V3: C1.1, C2.1, U1.28 (VDD), U1.8 (VDD)
- new net GND: C1.2, C2.2, U1.16 (AVSS), U1.31 (VSS), U1.43 (VSS), U1.7 (VSS)
